Commit message: 优化LW的模型

File: source/robot_lab/data/Robots/LW/LW_description/LW.urdf (robot description, URDF)
Before this commit: robot LW, 11 links, 10 joints
Links:
- link base_link: mass 10.76493269 -> 10.80229497
- link left_foot_link: mass 0.39895837 -> 0.44560421 
- link left_hip_link: mass 1.69532239 -> 1.72818563
- link left_shank_link: mass 1.97447981 -> 2.30578457
- link left_thigh_link: mass 2.08290871 -> 2.16887113 
- link left_wheel_link: mass 1.18607212 -> 1.22089955
- link right_foot_link: mass 0.39895837 -> 0.44560421
- link right_hip_link: mass 1.69532239 -> 1.72818563
- link right_shank_link: mass 1.97447981 -> 2.30578457
- link right_thigh_link: mass 2.08292210 -> 2.16888452
- link right_wheel_link: mass 1.18607212 -> 1.22089955
Joints:
- joint right_wheel_joint: origin xyz=-0.183850 -0.059500 -0.183850 rpy=0.000000 -0.000000 0.000000 -> xyz=-0.183850 -0.061000 -0.183850 rpy=0.000000 -0.000000 0.000000

Commit message: little fix

File: source/robot_lab/data/Robots/LW/LW_description/LW.urdf (robot description, URDF)
Before this commit: robot LW, 11 links, 10 joints
Links:
- link left_foot_link: mass 0.44560421  -> 0.44560421
- link left_thigh_link: mass 2.16887113  -> 2.16887113

Commit message: 2026-05-22

File: source/robot_lab/data/Robots/LW/LW_description/LW.urdf (robot description, URDF)
Before this commit: robot LW, 11 links, 10 joints
Links:
- link left_shank_link: mass 2.30578457 -> 2.40088457
- link right_shank_link: mass 2.30578457 -> 2.40088457
